File: kicad-bare-nrf52840/manufacturing/jlcpcb/source/parasite.kicad_sch (KiCad schematic)
At the start: 53 parts, among them J1 TC2030-SWD, Q1 MMBT3906, Q4 Q_Photo_NPN, SW1 B3U-1000P, U1 nRF52840-QIAA, U2 SHTC3, Y1 32.768kHz, Y2 32MHz

Commit message: feat: regenerate JLCPCB package for Kyocera Y2 substitution
Parts:
- Y2: Assembly_note Golledge custom MP12308 from Nordic reference; 32 MHz, CL 8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 -> 32 MHz fundamental, CL 8 pF, ESR 60 ohm max; +/-10 ppm init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; MPN MP12308 -> CX2016DB32000D0FLJCC; Manufacturer Golledge -> KYOCERA AVX; Source PCA10056 3.0.3 X1 -> DigiKey 478-CX2016DB32000D0FLJCCCT-ND
