File: kicad-bare-nrf52840/parasite.kicad_pcb (KiCad board)
At the start: 4 copper layers, 22 x 126.4 mm, 55 parts, among them J1 TC2030-SWD, Q1 MMBT3906, Q4 Q_Photo_NPN, SW1 B3U-1000P, U1 nRF52840-QIAA, U2 SHTC3, Y1 32.768kHz, Y2 32MHz

Commit message: feat: redesign for stocked antenna and capacitor with verified sensor ordering code
Parts:
- AE1: value 2450AT18B0100001E -> 2450AT18A0100001E
- C19: value 1.2p -> 1p
- C6: footprint Capacitor_SMD:C_0402_1005Metric -> Capacitor_SMD:C_0603_1608Metric
- L5: value 3.3n -> 3.9n
- moved C6 0.22 mm to (61.4, 45.4), turned to -90 degrees
Routing:
- net +3V0: track 94.6 -> 95.4 mm
- net GND: track 26.4 -> 25.7 mm
