File: kicad-large-smt-nrf52840/parasite.kicad_sch (KiCad schematic)
At the start: 53 parts, among them J1 TC2030-SWD, Q1 MMBT3906, Q4 Q_Photo_NPN, SW1 B3U-1000P, U1 nRF52840-QIAA, U2 SHTC3, Y1 32.768kHz, Y2 32MHz

Commit message: feat: enlarge ordinary passives and document approved package exceptions
Parts:
- C1: footprint Capacitor_SMD:C_0402_1005Metric -> Capacitor_SMD:C_1210_3225Metric; DigiKey 311-1036-1-ND -> (none); MPN CC0402KRX7R9BB102 -> (none); Manufacturer YAGEO -> (none); Package (none) -> 1210 imperial / 3225 metric; SelectionStatus (none) -> New package; purchasing MPN requires qualification
- C10, C2, C5, C8, C9: footprint Capacitor_SMD:C_0402_1005Metric -> Capacitor_SMD:C_1210_3225Metric; DigiKey 311-1338-1-ND -> (none); MPN CC0402KRX7R7BB104 -> (none); Manufacturer YAGEO -> (none); Package (none) -> 1210 imperial / 3225 metric; SelectionStatus (none) -> New package; purchasing MPN requires qualification
- C11, C7: footprint Capacitor_SMD:C_0402_1005Metric -> Capacitor_SMD:C_1210_3225Metric; LCSC C52923 -> (none); MPN CL05A105KA5NQNC -> (none); Manufacturer Samsung -> (none); Package (none) -> 1210 imperial / 3225 metric; SelectionStatus (none) -> New package; purchasing MPN requires qualification
- C12: footprint Capacitor_SMD:C_0402_1005Metric -> Capacitor_SMD:C_1210_3225Metric; DigiKey 311-1717-1-ND -> (none); MPN CC0402KRX7R8BB473 -> (none); Manufacturer YAGEO -> (none); Package (none) -> 1210 imperial / 3225 metric; SelectionStatus (none) -> New package; purchasing MPN requires qualification
- C13: footprint Capacitor_SMD:C_0402_1005Metric -> Capacitor_SMD:C_1210_3225Metric; DigiKey 311-1024-1-ND -> (none); MPN CC0402JRNPO9BN101 -> (none); Manufacturer YAGEO -> (none); Package (none) -> 1210 imperial / 3225 metric; SelectionStatus (none) -> New package; purchasing MPN requires qualification
- C14, C15, C3, C4: footprint Capacitor_SMD:C_0402_1005Metric -> Capacitor_SMD:C_1210_3225Metric; DigiKey 311-1016-1-ND -> (none); MPN CC0402JRNPO9BN120 -> (none); Manufacturer YAGEO -> (none); Package (none) -> 1210 imperial / 3225 metric; SelectionStatus (none) -> New package; purchasing MPN requires qualification
- C16: footprint Capacitor_SMD:C_0402_1005Metric -> Capacitor_SMD:C_1210_3225Metric; LCSC C307452 -> (none); MPN CL05C821JB5NNNC -> (none); Manufacturer Samsung -> (none); Package (none) -> 1210 imperial / 3225 metric; SelectionStatus (none) -> New package; purchasing MPN requires qualification
- C6: footprint Capacitor_SMD:C_0603_1608Metric -> Capacitor_SMD:C_1210_3225Metric; DigiKey 490-GRM188R61C475KE11JCT-ND -> (none); MPN GRM188R61C475KE11J -> (none); Manufacturer Murata -> (none); Package (none) -> 1210 imperial / 3225 metric; SelectionStatus (none) -> New package; purchasing MPN requires qualification
- D2: footprint LED_SMD:LED_0603_1608Metric -> LED_SMD:LED_PLCC-2_3.4x3.0mm_KA; DigiKey 160-1436-1-ND -> (none); MPN LTST-C190KRKT -> VLMR334BACB-GS08; Manufacturer Lite-On -> Vishay; Package (none) -> PLCC-2; SelectionStatus (none) -> Red LED; keep 1k current limiting resistor; verify low-curr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
- L1: footprint Inductor_SMD:L_0603_1608Metric -> Inductor_SMD:L_Bourns-SRN4018; LCSC C2047264 -> (none); MPN MLZ1608M100WTD25 -> SRN4018-100M; Manufacturer TDK -> Bourns; Package (none) -> 4.0 x 4.0 mm; SelectionStatus (none) -> Prototype candidate; converter efficiency requires verifica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
- L2: footprint Inductor_SMD:L_0402_1005Metric -> Inductor_SMD:L_Coilcraft_1008HQ_2520Metric; LCSC C86059 -> (none); MPN LQG15HS15NJ02D -> 1008CS-150XJRC; Manufacturer Murata -> Coilcraft; Package (none) -> 1008 imperial; 2.92 x 2.79 mm max; SelectionStatus (none) -> 1008CS uses matching 1008HQ land geometry; prototype filter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
- R1, R4, R7, R8: footprint Resistor_SMD:R_0402_1005Metric -> Resistor_SMD:R_1210_3225Metric; DigiKey 311-10.0KLRCT-ND -> (none); MPN RC0402FR-0710KL -> RC1210FR-0710KL; Package (none) -> 1210 imperial / 3225 metric; Power (none) -> 0.5W; SelectionStatus (none) -> 1210 1% resistor; stock not checked
- R10: footprint Resistor_SMD:R_0402_1005Metric -> Resistor_SMD:R_1210_3225Metric; DigiKey 311-470LRCT-ND -> (none); MPN RC0402FR-07470RL -> RC1210FR-07470RL; Package (none) -> 1210 imperial / 3225 metric; Power (none) -> 0.5W; SelectionStatus (none) -> 1210 1% resistor; stock not checked
- R2: footprint Resistor_SMD:R_0402_1005Metric -> Resistor_SMD:R_1210_3225Metric; DigiKey 311-1.00KLRCT-ND -> (none); MPN RC0402FR-071KL -> RC1210FR-071KL; Package (none) -> 1210 imperial / 3225 metric; Power (none) -> 0.5W; SelectionStatus (none) -> 1210 1% resistor; stock not checked
- R6: footprint Resistor_SMD:R_0402_1005Metric -> Resistor_SMD:R_1210_3225Metric; DigiKey 311-1.00MLRCT-ND -> (none); MPN RC0402FR-071ML -> RC1210FR-071ML; Package (none) -> 1210 imperial / 3225 metric; Power (none) -> 0.5W; SelectionStatus (none) -> 1210 1% resistor; stock not checked
