File: kicad-raytac-plant-monitor/parasite.kicad_sch (KiCad schematic)
At the start: 53 parts, among them J1 TC2030-SWD, Q1 MMBT3906, Q4 Q_Photo_NPN, SW1 B3U-1000P, U1 nRF52840-QIAA, U2 SHTC3, Y1 32.768kHz, Y2 32MHz

Commit message: feat: replace bare MCU with Raytac module and add debug I2C NFC interfaces
Parts:
- removed AE1: 2450AT18A0100001E, RF_Antenna:Johanson_2450AT18x100, symbol Device:Antenna_Chip
- removed C10, C8, C9: 100n, Capacitor_SMD:C_1210_3225Metric, symbol Device:C_Small
- removed C11, C7: 1u, Capacitor_SMD:C_1210_3225Metric, symbol Device:C_Small
- removed C12: 47n, Capacitor_SMD:C_1210_3225Metric, symbol Device:C_Small
- removed C13: 100p, Capacitor_SMD:C_1210_3225Metric, symbol Device:C_Small
- removed C14, C15: 12p, Capacitor_SMD:C_1210_3225Metric, symbol Device:C_Small
- removed C16: 820p, Capacitor_SMD:C_1210_3225Metric, symbol Device:C_Small
- removed C17: 0.8p, Capacitor_SMD:C_0402_1005Metric, symbol Device:C_Small
- removed C18: 0.5p, Capacitor_SMD:C_0402_1005Metric, symbol Device:C_Small
- removed C19: 1p, Capacitor_SMD:C_0402_1005Metric, symbol Device:C_Small
- removed J1: TC2030-SWD, Connector:Tag-Connect_TC2030-IDC-NL_2x03_P1.27mm_Vertical, symbol Connector_Generic:Conn_02x03_Odd_Even
- removed L1: 10u, Inductor_SMD:L_Bourns-SRN4018, symbol Device:L
- removed L2: 15n, Inductor_SMD:L_Coilcraft_1008HQ_2520Metric, symbol Device:L
- removed L3: 4.7n, Inductor_SMD:L_0402_1005Metric, symbol Device:L
- removed L4: 2.7n, Inductor_SMD:L_0402_1005Metric, symbol Device:L
- removed L5: 3.9n, Inductor_SMD:L_0402_1005Metric, symbol Device:L
- removed TP8: 0.10, TestPoint:TestPoint_Pad_D1.0mm, symbol Connector:TestPoint
- removed U1: nRF52840-QIAA, Package_DFN_QFN:Nordic_AQFN-73-1EP_7x7mm_P0.5mm, symbol MCU_Nordic:nRF52840
- removed Y2: 32MHz, Crystal:Crystal_SMD_2016-4Pin_2.0x1.6mm, symbol Device:Crystal_GND24
- added J1: Cortex SWD 10-pin, Connector_PinHeader_1.27mm:PinHeader_2x05_P1.27mm_Vertical_SMD, symbol Connector:Conn_ARM_JTAG_SWD_10
- added J2: I2C 3V, Connector_PinHeader_2.54mm:PinHeader_1x04_P2.54mm_Vertical, symbol Connector_Generic:Conn_01x04
- added J3: NFC ANTENNA, Connector_PinHeader_2.54mm:PinHeader_1x02_P2.54mm_Vertical, symbol Connector_Generic:Conn_01x02
- added U1: MDBT50Q-1MV2, RF_Module:Raytac_MDBT50Q, symbol RF_Module:MDBT50Q-1MV2
- C5: Dielectric (none) -> X7R; Package 1210 imperial / 3225 metric -> (none); SelectionStatus New package; purchasing MPN requires qualification -> (none); Voltage (none) -> 50V
- C6: value 4.7u -> 10u; Assembly_note Larger 0603 bulk capacitor. Typical effective capacitance a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 -> (none); Dielectric X5R -> X7R; Package 1210 imperial / 3225 metric -> (none); SelectionStatus New package; purchasing MPN requires qualification -> (none); Tolerance 10% -> (none)
Connections:
- net DEC1 is gone; now on net +3V0: C5.1
- net +3V0: now also J1.1 (VTref), J2.1 (Pin_1), U1.28 (VDD), U1.30 (VDDH)
- net BTN1: now also U1.14 (P0.30)
- net GND: now also J1.3 (GND), J1.5 (GND), J1.9 (GNDDetect), J2.2 (Pin_2), U1.1 (GND), U1.15 (GND), U1.2 (GND), U1.32 (VBUS), U1.33 (GND), U1.55 (GND)
- net LED: now also U1.13 (P0.28)
- net PHOTO_OUT: now also U1.11 (P0.02)
- net PHOTO_V: now also U1.10 (P0.29)
- net PWM: now also U1.21 (P0.05)
- net RST: now also J1.10 (~{RESET}), U1.40 (P0.18)
- net SCL: now also J2.4 (Pin_4), U1.37 (P0.13)
- net SDA: now also J2.3 (Pin_3), U1.48 (P0.24)
- net SENS_OUT: now also U1.9 (P0.03)
- net SWDCLK: now also J1.4 (SWCLK/TCK), U1.53 (SWDCLK)
- net SWDIO: now also J1.2 (SWDIO/TMS), U1.51 (SWDIO)
- net XL1: now also U1.17 (P0.00)
- net XL2: now also U1.18 (P0.01)
- new net NFC1: J3.1 (Pin_1), U1.52 (P0.09)
- new net NFC2: J3.2 (Pin_2), U1.54 (P0.10)
- new net SWO: J1.6 (SWO/TDO), U1.47 (P1.00)
- no-connect marks 44 -> 40
Other:
- title: b-parasite — bare nRF52840 -> BLE Plant Monitor - Raytac MDBT50Q-1MV2

Commit message: feat: compact Raytac monitor with 0805 passives and straight 30 mm sides
Parts:
- C1: footprint Capacitor_SMD:C_1210_3225Metric -> Capacitor_SMD:C_0805_2012Metric; Dielectric (none) -> C0G; MPN (none) -> C0805C102J5GACTU; Manufacturer (none) -> KEMET; Package 1210 imperial / 3225 metric -> 0805; SelectionStatus New package; purchasing MPN requires qualification -> 0805; specified electrical value; inventory not checked; Voltage (none) -> 50V
- C2: footprint Capacitor_SMD:C_1210_3225Metric -> Capacitor_SMD:C_0805_2012Metric; Dielectric (none) -> X7R; MPN (none) -> C0805C104K5RACTU; Manufacturer (none) -> KEMET; Package 1210 imperial / 3225 metric -> 0805; SelectionStatus New package; purchasing MPN requires qualification -> 0805; specified electrical value; inventory not checked; Voltage (none) -> 50V
- C3, C4: footprint Capacitor_SMD:C_1210_3225Metric -> Capacitor_SMD:C_0805_2012Metric; Dielectric (none) -> C0G; MPN (none) -> C0805C120J5GACTU; Manufacturer (none) -> KEMET; Package 1210 imperial / 3225 metric -> 0805; SelectionStatus New package; purchasing MPN requires qualification -> 0805; specified electrical value; inventory not checked; Voltage (none) -> 50V
- C5: footprint Capacitor_SMD:C_1210_3225Metric -> Capacitor_SMD:C_0805_2012Metric; MPN (none) -> C0805C104K5RACTU; Manufacturer (none) -> KEMET; Package (none) -> 0805; SelectionStatus (none) -> 0805; specified electrical value; inventory not checked
- C6: footprint Capacitor_SMD:C_1210_3225Metric -> Capacitor_SMD:C_0805_2012Metric; Dielectric X7R -> X5R; MPN (none) -> GRM21BR61C106KE15L; Manufacturer (none) -> Murata; Package (none) -> 0805; SelectionStatus (none) -> 0805; specified electrical value; inventory not checked
- D2: footprint LED_SMD:LED_PLCC-2_3.4x3.0mm_KA -> LED_SMD:LED_0805_2012Metric; MPN VLMR334BACB-GS08 -> AP2012SURCK; Manufacturer Vishay -> Kingbright; Package PLCC-2 -> 0805
- R1, R4, R7, R8: footprint Resistor_SMD:R_1210_3225Metric -> Resistor_SMD:R_0805_2012Metric; MPN RC1210FR-0710KL -> RC0805FR-0710KL; Package 1210 imperial / 3225 metric -> 0805; Power 0.5W -> 0.125W; SelectionStatus 1210 1% resistor; stock not checked -> 0805 1% resistor; inventory not checked
- R10: footprint Resistor_SMD:R_1210_3225Metric -> Resistor_SMD:R_0805_2012Metric; MPN RC1210FR-07470RL -> RC0805FR-07470RL; Package 1210 imperial / 3225 metric -> 0805; Power 0.5W -> 0.125W; SelectionStatus 1210 1% resistor; stock not checked -> 0805 1% resistor; inventory not checked
- R2: footprint Resistor_SMD:R_1210_3225Metric -> Resistor_SMD:R_0805_2012Metric; MPN RC1210FR-071KL -> RC0805FR-071KL; Package 1210 imperial / 3225 metric -> 0805; Power 0.5W -> 0.125W; SelectionStatus 1210 1% resistor; stock not checked -> 0805 1% resistor; inventory not checked
- R6: footprint Resistor_SMD:R_1210_3225Metric -> Resistor_SMD:R_0805_2012Metric; MPN RC1210FR-071ML -> RC0805FR-071ML; Package 1210 imperial / 3225 metric -> 0805; Power 0.5W -> 0.125W; SelectionStatus 1210 1% resistor; stock not checked -> 0805 1% resistor; inventory not checked
