File: kicad-raytac-plant-monitor/parasite.kicad_pcb (KiCad board)
At the start: 4 copper layers, 30 x 126.4 mm, 36 parts, among them J1 Cortex SWD 10-pin, J2 I2C 3V, J3 NFC ANTENNA, Q1 MMBT3906, Q4 Q_Photo_NPN, SW1 B3U-1000P, U1 MDBT50Q-1MV2, U2 SHTC3, Y1 32.768kHz

Commit message: feat: add pointed Raytac probe and stitch its ground pours
Routing:
- net GND: vias 8 -> 9
Other:
- outline, holes or cut-outs redrawn
Changed lines of the file:
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@@
 		(layer "B.SilkS")
 	)
-	(gr_rect
+	(gr_line
 		(start 53 27)
-		(end 83 153.4)
+		(end 83 27)
 		(stroke
 			(width 0.05)
 			(type default)
 		)
-		(fill no)
+		(layer "Edge.Cuts")
+	)
+	(gr_line
+		(start 53 138.4)
+		(end 53 27)
+		(stroke
+			(width 0.05)
+			(type default)
+		)
+		(layer "Edge.Cuts")
+	)
+	(gr_line
+		(start 68 153.4)
+		(end 53 138.4)
+		(stroke
+			(width 0.05)
+			(type default)
+		)
+		(layer "Edge.Cuts")
+	)
+	(gr_line
+		(start 83 27)
+		(end 83 138.4)
+		(stroke
+			(width 0.05)
+			(type default)
+		)
+		(layer "Edge.Cuts")
+	)
+	(gr_line
+		(start 83 138.4)
+		(end 68 153.4)
+		(stroke
+			(width 0.05)
+			(type default)
+		)
 		(layer "Edge.Cuts")
 	)
@@
 		(size 0.6)
 		(drill 0.3)
+		(layers "F.Cu" "B.Cu")
+		(net "GND")
+	)
+	(via
+		(at 68 150.5)
+		(size 0.6)
+		(drill 0.3)
